File: Design Files/Auto-UPDI-with-switch.kicad_pcb (KiCad board)
At the start: 2 copper layers, 27.3 x 24.1 mm, 5 parts, among them J1 1x06_P2.54mm_Horizontal_SMD, J2 1x06 Pin header 2.54 SMD, SW1 Switch_Slide_RightAngle_CnK

Commit message: added files and updated readme
Parts:
- renumbered D5 to D1, R4 to R1
Connections:
- J1 pad 6: DTR -> unconnected-(J1-Pad6)
Changed lines of the file:
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@@
 	(net 4 "VCC")
 	(net 5 "RX")
-	(net 6 "DTR")
+	(net 6 "unconnected-(J1-Pad6)")
 	(net 7 "UPDI")
 	(net 8 "T-RX")
@@
 			(size 2.5 1.7)
 			(layers "F.Cu" "F.Mask" "F.Paste")
-			(net 6 "DTR")
-			(pintype "passive")
+			(net 6 "unconnected-(J1-Pad6)")
+			(pintype "passive+no_connect")
 		)
 		(embedded_fonts no)
@@
 		(tags "switch spdt right angle slide")
 		(property "Reference" "SW1"
-			(at 0 -4.3 0)
+			(at -3.4925 -4.3 0)
 			(layer "F.SilkS")
 			(effects
@@
 		)
 		(embedded_fonts no)
-		(model "${KISYS3DMOD}/Buttons_Switches_SMD.3dshapes/SW_SPDT_CK-JS102011SAQN.wrl"
+		(model "C:/kicad/libraries/kicad/fab.3dshapes/AYZ0102AGRLC.stp"
 			(offset
 				(xyz 0 0 0)
@@
 			)
 			(rotate
-				(xyz 0 0 0)
+				(xyz -90 -0 -0)
 			)
 		)
@@
 		(tags "horizontal pin header SMD 2.54mm")
 		(property "Reference" "J2"
-			(at 3.73 6.3 180)
+			(at 4.365 6.3 180)
 			(layer "F.SilkS")
 			(effects
@@
 		)
 		(embedded_fonts no)
+		(model "C:/kicad/libraries/kicad/fab.3dshapes/PinSocket-01x06_P2.54mm_Horizontal_SMD.step"
+			(offset
+				(xyz 0 0 0)
+			)
+			(scale
+				(xyz 1 1 1)
+			)
+			(rotate
+				(xyz 0 0 0)
+			)
+		)
 	)
 	(footprint "fab:Diode_Schottky_MiniSMA"
@@
 		(descr "Mini-SMA  Schottky diode footprint")
 		(tags "Mini-SMA schottky diode")
-		(property "Reference" "D5"
-			(at 0 0 0)
+		(property "Reference" "D1"
+			(at 1.905 1.905 0)
 			(layer "F.SilkS")
 			(effects
@@
 		(sheetname "/")
 		(sheetfile "Auto-UPDI-with-switch.kicad_sch")
-		(attr through_hole)
+		(attr smd)
 		(fp_line
 			(start -1.75 1.25)
@@
 		)
 		(embedded_fonts no)
+		(model "C:/kicad/libraries/kicad/fab.3dshapes/Diode-Schottky-SOD123.step"
+			(offset
+				(xyz 0 0 0.7)
+			)
+			(scale
+				(xyz 1 1 1)
+			)
+			(rotate
+				(xyz -90 -0 -0)
+			)
+		)
 	)
 	(footprint "fab:R_1206"
@@
 		(descr "Resistor SMD 1206, hand soldering")
 		(tags "resistor 1206")
-		(property "Reference" "R4"
-			(at 0 0 0)
-			(layer "F.SilkS")
-			(effects
+		(property "Reference" "R1"
+			(at -1.905 -1.905 0)
+			(layer "F.SilkS")
+			(effects
