File: Design Files/Auto-UPDI-with-switch.kicad_sch (KiCad schematic)
At the start: 5 parts, among them J1 1x06_P2.54mm_Horizontal_SMD, J2 1x06 Pin header 2.54 SMD, SW1 Switch_Slide_RightAngle_CnK

Commit message: added files and updated readme
Parts:
- renumbered D5 to D1, R4 to R1
Other:
- note added: "6pin FTDI header for Target board"
- note added: "6pin FTDI pin for the FTDI converter"
- note added: "FTDI to UPDI Circuit"
- note added: "UPDI/UART Selcetion Switch"
- company: (none) -> Designed by Saheen palayi | Super Fablab Kerala
- title: (none) -> UPDI/UART Switch
- moved on the sheet: D1, J1, J2, R1, SW1
